Commit message: Add files via upload

File: src/dual_description/urdf/robot_table.urdf (robot description, URDF)
Before this commit: robot robot_table, 6 links, 5 joints
Links:
- link table_base_hong: geometry visual box size=1.2 1.8 0.75
- link table_base_kong: geometry visual box size=1.2 1.8 0.75
- link table_middle: geometry visual box size=0.8 1.2 0.705
- link upper_block_hong: geometry visual box size=0.25 0.25 0.02
- link upper_block_kong: geometry visual box size=0.25 0.25 0.02
Joints:
- joint table_to_block_hong: origin xyz=0.7 0 0.75 rpy=0 0 0 -> xyz=0.465 0 0.75 rpy=0 0 0
- joint table_to_block_kong: origin xyz=-0.7 0 0.75 rpy=0 0 0 -> xyz=-0.465 0 0.75 rpy=0 0 0
- joint world_to_table_hong: origin xyz=-2 0 0 rpy=0 0 0 -> xyz=-1.35 0 0 rpy=0 0 0
- joint world_to_table_kong: origin xyz=2 0 0 rpy=0 0 0 -> xyz=1.35 0 0 rpy=0 0 0
