Commit message: Add files via upload

File: src/dual_description/urdf/soft_hybrid_gripper2_URDF.urdf (robot description, URDF)
Before this commit: robot soft hybrid gripper URDF, 4 links, 3 joints
Links:
- removed link base_link2
- removed link rigid_link2
- removed link rigid_tip_link2
- removed link soft_tip_link2
- added link base_link1, mass 0.117842634947847; collision mesh filename=package://dual_description/meshes/base_link1.STL; visual mesh filename=package://dual_description/meshes/base_link1.STL
- added link rigid_link1, mass 0.0445322519868914; collision mesh filename=package://dual_description/meshes/rigid_link.STL; visual mesh filename=package://dual_description/meshes/rigid_link.STL
- added link rigid_tip_link1, mass 0.0134476259243688; collision mesh filename=package://dual_description/meshes/rigid_tip_link.STL; visual mesh filename=package://dual_description/meshes/rigid_tip_link.STL
- added link soft_tip_link1, mass 0.0267549348618611; collision mesh filename=package://dual_description/meshes/soft_tip_link.STL; visual mesh filename=package://dual_description/meshes/soft_tip_link.STL
Joints:
- removed joint rigid_rev_joint2
- removed joint rigid_tip_joint2
- removed joint soft_tip_joint2
- added joint rigid_rev_joint1: type revolute, parent base_link1, child rigid_link1, origin xyz=-0.018 0.0604 0.031 rpy=0 0 0, axis 0 -1 0, limit lower=0 upper=0 effort=0 velocity=0
- added joint rigid_tip_joint1: type continuous, parent rigid_link1, child rigid_tip_link1, origin xyz=0.029389 -0.00085 0.11906 rpy=0 -0.13252 -3.1416, axis 0 1 0
- added joint soft_tip_joint1: type fixed, parent base_link1, child soft_tip_link1, origin xyz=0.11681 0.061 0.098742 rpy=0 -0.66549 0, axis 0 0 0

Commit message: Add files via upload

File: src/dual_description/urdf/soft_hybrid_gripper2_URDF.urdf (robot description, URDF)
Before this commit: robot soft hybrid gripper URDF, 4 links, 3 joints
Joints:
- joint rigid_rev_joint1: limit lower=0 upper=0 effort=0 velocity=0 -> lower=${-pi} upper=${pi} effort=0 velocity=0; type revolute -> continuous

File: src/dual_description/urdf/soft_hybrid_gripper_URDF.urdf (robot description, URDF)
Before this commit: robot soft hybrid gripper URDF, 4 links, 3 joints
Joints:
- joint rigid_rev_joint2: limit lower=0 upper=0 effort=0 velocity=0 -> lower=${-pi} upper=${pi} effort=0 velocity=0; type revolute -> continuous

Commit message: Add files via upload
Update soft_hybrid_gripper_URDF2.urdf, and soft_hybrid_gripper_URDF.urdf. Enable two continuous joints and disabled two joints.

File: src/dual_description/urdf/soft_hybrid_gripper2_URDF.urdf (robot description, URDF)
Before this commit: robot soft hybrid gripper URDF, 4 links, 3 joints
Joints:
- joint rigid_tip_joint1: type continuous -> fixed

File: src/dual_description/urdf/soft_hybrid_gripper_URDF.urdf (robot description, URDF)
Before this commit: robot soft hybrid gripper URDF, 4 links, 3 joints
Joints:
- joint rigid_tip_joint2: type continuous -> fixed
