Commit message: Add files via upload

File: src/ur10/liwei_ur_description/urdf/ur10.urdf.xacro (robot description, xacro)
@@ -50,5 +50,5 @@
     <xacro:property name="elbow_offset" value="0.049042" /> <!-- measured from model -->
     <xacro:property name="upper_arm_inertia_offset" value="0.175" />  <!-- measured from model -->
-    <!-- This is for compatibility reasons, as transformation between base and base_link was always 180 degree in the ur_description -->
+    <!-- This is for compatibility reasons, as transformation between base and base_link was always 180 degree in the liwei_ur_description -->
     <xacro:property name="base_correction" value="${pi}" />
     <link name="${prefix}base_link" >
@@ -56,5 +56,5 @@
         <origin xyz="0 0 0" rpy="0 0 ${base_correction}"/>
         <geometry>
-          <mesh filename="package://ur_description/meshes/ur10/visual/base.dae"/>
+          <mesh filename="package://liwei_ur_description/meshes/ur10/visual/base.dae"/>
         </geometry>
         <material name="LightGrey">
@@ -65,5 +65,5 @@
         <origin xyz="0 0 0" rpy="0 0 ${base_correction}"/>
         <geometry>
-          <mesh filename="package://ur_description/meshes/ur10/collision/base.stl"/>
+          <mesh filename="package://liwei_ur_description/meshes/ur10/collision/base.stl"/>
         </geometry>
       </collision>
@@ -95,5 +95,5 @@
         <origin xyz="0 0 0" rpy="0 0 ${pi}"/>
         <geometry>
-          <mesh filename="package://ur_description/meshes/ur10/visual/shoulder.dae"/>
+          <mesh filename="package://liwei_ur_description/meshes/ur10/visual/shoulder.dae"/>
         </geometry>
         <material name="LightGrey">
@@ -104,5 +104,5 @@
         <origin xyz="0 0 0" rpy="0 0 ${pi}"/>
         <geometry>
-          <mesh filename="package://ur_description/meshes/ur10/collision/shoulder.stl"/>
+          <mesh filename="package://liwei_ur_description/meshes/ur10/collision/shoulder.stl"/>
         </geometry>
       </collision>
@@ -134,5 +134,5 @@
         <origin xyz="0 0 ${shoulder_offset}" rpy="${pi/2} 0 ${-pi/2}"/>
         <geometry>
-          <mesh filename="package://ur_description/meshes/ur10/visual/upperarm.dae"/>
+          <mesh filename="package://liwei_ur_description/meshes/ur10/visual/upperarm.dae"/>
         </geometry>
         <material name="LightGrey">
@@ -143,5 +143,5 @@
         <origin xyz="0 0 ${shoulder_offset}" rpy="${pi/2} 0 ${-pi/2}"/>
         <geometry>
-          <mesh filename="package://ur_description/meshes/ur10/collision/upperarm.stl"/>
+          <mesh filename="package://liwei_ur_description/meshes/ur10/collision/upperarm.stl"/>
         </geometry>
       </collision>
@@ -173,5 +173,5 @@
         <origin xyz="0 0 ${elbow_offset}" rpy="${pi/2} 0 ${-pi/2}"/>
         <geometry>
-          <mesh filename="package://ur_description/meshes/ur10/visual/forearm.dae"/>
+          <mesh filename="package://liwei_ur_description/meshes/ur10/visual/forearm.dae"/>
         </geometry>
         <material name="LightGrey">
@@ -182,5 +182,5 @@
         <origin xyz="0 0 ${elbow_offset}" rpy="${pi/2} 0 ${-pi/2}"/>
         <geometry>
-          <mesh filename="package://ur_description/meshes/ur10/collision/forearm.stl"/>
+          <mesh filename="package://liwei_ur_description/meshes/ur10/collision/forearm.stl"/>
         </geometry>
       </collision>
@@ -212,5 +212,5 @@
         <origin xyz="0 0 -0.1149" rpy="${pi/2} 0 0"/>
         <geometry>
-          <mesh filename="package://ur_description/meshes/ur10/visual/wrist1.dae"/>
+          <mesh filename="package://liwei_ur_description/meshes/ur10/visual/wrist1.dae"/>
         </geometry>
         <material name="LightGrey">
@@ -221,5 +221,5 @@
         <origin xyz="0 0 -0.1149" rpy="${pi/2} 0 0"/>
         <geometry>
-          <mesh filename="package://ur_description/meshes/ur10/collision/wrist1.stl"/>
+          <mesh filename="package://liwei_ur_description/meshes/ur10/collision/wrist1.stl"/>
         </geometry>
       </collision>
@@ -251,5 +251,5 @@
         <origin xyz="0 0 -0.1158" rpy="0 0 0"/>
         <geometry>
-          <mesh filename="package://ur_description/meshes/ur10/visual/wrist2.dae"/>
+          <mesh filename="package://liwei_ur_description/meshes/ur10/visual/wrist2.dae"/>
         </geometry>
         <material name="LightGrey">
@@ -260,5 +260,5 @@
         <origin xyz="0 0 -0.1158" rpy="0 0 0"/>
         <geometry>
-          <mesh filename="package://ur_description/meshes/ur10/collision/wrist2.stl"/>
+          <mesh filename="package://liwei_ur_description/meshes/ur10/collision/wrist2.stl"/>
         </geometry>
       </collision>
@@ -290,5 +290,5 @@
         <origin xyz="0 0 -0.0922" rpy="${pi/2} 0 0"/>
         <geometry>
-          <mesh filename="package://ur_description/meshes/ur10/visual/wrist3.dae"/>
+          <mesh filename="package://liwei_ur_description/meshes/ur10/visual/wrist3.dae"/>
         </geometry>
         <material name="LightGrey">
@@ -299,5 +299,5 @@
         <origin xyz="0 0 -0.0922" rpy="${pi/2} 0 0"/>
         <geometry>
-          <mesh filename="package://ur_description/meshes/ur10/collision/wrist3.stl"/>
+          <mesh filename="package://liwei_ur_description/meshes/ur10/collision/wrist3.stl"/>
         </geometry>
       </collision>

File: src/ur10/liwei_ur_description/urdf/ur10_kong.urdf.xacro (robot description, xacro)
@@ -50,5 +50,5 @@
     <xacro:property name="elbow_offset" value="0.049042" /> <!-- measured from model -->
     <xacro:property name="upper_arm_inertia_offset" value="0.175" />  <!-- measured from model -->
-    <!-- This is for compatibility reasons, as transformation between base and base_link was always 180 degree in the ur_description -->
+    <!-- This is for compatibility reasons, as transformation between base and base_link was always 180 degree in the liwei_ur_description -->
     <xacro:property name="base_correction" value="${pi}" />
     <link name="${prefix}base_link" >
@@ -56,5 +56,5 @@
         <origin xyz="0 0 0" rpy="0 0 ${base_correction}"/>
         <geometry>
-          <mesh filename="package://ur_description/meshes/ur10/visual/base.dae"/>
+          <mesh filename="package://liwei_ur_description/meshes/ur10/visual/base.dae"/>
         </geometry>
         <material name="LightGrey">
@@ -65,5 +65,5 @@
         <origin xyz="0 0 0" rpy="0 0 ${base_correction}"/>
         <geometry>
-          <mesh filename="package://ur_description/meshes/ur10/collision/base.stl"/>
+          <mesh filename="package://liwei_ur_description/meshes/ur10/collision/base.stl"/>
         </geometry>
       </collision>
@@ -95,5 +95,5 @@
         <origin xyz="0 0 0" rpy="0 0 ${pi}"/>
         <geometry>
-          <mesh filename="package://ur_description/meshes/ur10/visual/shoulder.dae"/>
+          <mesh filename="package://liwei_ur_description/meshes/ur10/visual/shoulder.dae"/>
         </geometry>
         <material name="LightGrey">
@@ -104,5 +104,5 @@
         <origin xyz="0 0 0" rpy="0 0 ${pi}"/>
         <geometry>
-          <mesh filename="package://ur_description/meshes/ur10/collision/shoulder.stl"/>
+          <mesh filename="package://liwei_ur_description/meshes/ur10/collision/shoulder.stl"/>
         </geometry>
       </collision>
@@ -134,5 +134,5 @@
         <origin xyz="0 0 ${shoulder_offset}" rpy="${pi/2} 0 ${-pi/2}"/>
         <geometry>
-          <mesh filename="package://ur_description/meshes/ur10/visual/upperarm.dae"/>
+          <mesh filename="package://liwei_ur_description/meshes/ur10/visual/upperarm.dae"/>
         </geometry>
         <material name="LightGrey">
@@ -143,5 +143,5 @@
         <origin xyz="0 0 ${shoulder_offset}" rpy="${pi/2} 0 ${-pi/2}"/>
         <geometry>
-          <mesh filename="package://ur_description/meshes/ur10/collision/upperarm.stl"/>
+          <mesh filename="package://liwei_ur_description/meshes/ur10/collision/upperarm.stl"/>
         </geometry>
       </collision>
@@ -173,5 +173,5 @@
         <origin xyz="0 0 ${elbow_offset}" rpy="${pi/2} 0 ${-pi/2}"/>
         <geometry>
-          <mesh filename="package://ur_description/meshes/ur10/visual/forearm.dae"/>
+          <mesh filename="package://liwei_ur_description/meshes/ur10/visual/forearm.dae"/>
         </geometry>
         <material name="LightGrey">
@@ -182,5 +182,5 @@
         <origin xyz="0 0 ${elbow_offset}" rpy="${pi/2} 0 ${-pi/2}"/>
         <geometry>
-          <mesh filename="package://ur_description/meshes/ur10/collision/forearm.stl"/>
+          <mesh filename="package://liwei_ur_description/meshes/ur10/collision/forearm.stl"/>
         </geometry>
       </collision>
@@ -212,5 +212,5 @@
         <origin xyz="0 0 -0.1149" rpy="${pi/2} 0 0"/>
         <geometry>
-          <mesh filename="package://ur_description/meshes/ur10/visual/wrist1.dae"/>
+          <mesh filename="package://liwei_ur_description/meshes/ur10/visual/wrist1.dae"/>
         </geometry>
         <material name="LightGrey">
@@ -221,5 +221,5 @@
         <origin xyz="0 0 -0.1149" rpy="${pi/2} 0 0"/>
         <geometry>
-          <mesh filename="package://ur_description/meshes/ur10/collision/wrist1.stl"/>
+          <mesh filename="package://liwei_ur_description/meshes/ur10/collision/wrist1.stl"/>
         </geometry>
       </collision>
@@ -251,5 +251,5 @@
         <origin xyz="0 0 -0.1158" rpy="0 0 0"/>
         <geometry>
-          <mesh filename="package://ur_description/meshes/ur10/visual/wrist2.dae"/>
+          <mesh filename="package://liwei_ur_description/meshes/ur10/visual/wrist2.dae"/>
         </geometry>
         <material name="LightGrey">
@@ -260,5 +260,5 @@
         <origin xyz="0 0 -0.1158" rpy="0 0 0"/>
         <geometry>
-          <mesh filename="package://ur_description/meshes/ur10/collision/wrist2.stl"/>
+          <mesh filename="package://liwei_ur_description/meshes/ur10/collision/wrist2.stl"/>
         </geometry>
       </collision>
@@ -290,5 +290,5 @@
         <origin xyz="0 0 -0.0922" rpy="${pi/2} 0 0"/>
         <geometry>
-          <mesh filename="package://ur_description/meshes/ur10/visual/wrist3.dae"/>
+          <mesh filename="package://liwei_ur_description/meshes/ur10/visual/wrist3.dae"/>
         </geometry>
         <material name="LightGrey">
@@ -299,5 +299,5 @@
         <origin xyz="0 0 -0.0922" rpy="${pi/2} 0 0"/>
         <geometry>
-          <mesh filename="package://ur_description/meshes/ur10/collision/wrist3.stl"/>
+          <mesh filename="package://liwei_ur_description/meshes/ur10/collision/wrist3.stl"/>
         </geometry>
       </collision>
